Commit message: Update sim2sim
修改sim2sim配置,将x2_urdf的ankle_pitch碰撞删除,调整armature与mujoco保持一致

File: source/whole_body_tracking/whole_body_tracking/assets/x2_ultra/x2_ultra.urdf (robot description, URDF)
Before this commit: robot x2t2.5, 41 links, 40 joints
Links:
- link left_ankle_pitch_link: geometry visual mesh filename=./meshes/left_ankle_pitch_link.STL
- link right_ankle_pitch_link: geometry visual mesh filename=./meshes/right_ankle_pitch_link.STL
