Commit message: updare simple_collision
新增简易urdf,将wrist
_roll作为跟踪目标,添加所有lafan1 pkl文件

File: source/whole_body_tracking/whole_body_tracking/assets/x2_ultra/x2_ultra_simple_collision.urdf (robot description, URDF)
Before this commit: robot x2t2.5, 41 links, 40 joints
Links:
- removed link base_link
- removed link lidar_chest_front
- link head_pitch_link: geometry visual mesh filename=./meshes/head_pitch_link.STL
- link head_yaw_link: geometry visual mesh filename=./meshes/head_yaw_link.STL
- link left_ankle_pitch_link: geometry visual mesh filename=./meshes/left_ankle_pitch_link.STL
- link left_ankle_roll_link: geometry collision sphere radius=0.005; collision sphere radius=0.005
- link left_elbow_link: geometry collision cylinder length=0.09 radius=0.04; visual mesh filename=./meshes/left_elbow_link.STL
- link left_hip_pitch_link: geometry visual mesh filename=./meshes/left_hip_pitch_link.STL
- link left_hip_yaw_link: geometry collision cylinder length=0.03 radius=0.042; collision cylinder length=0.03 radius=0.042
- link left_shoulder_pitch_link: geometry visual mesh filename=./meshes/left_shoulder_pitch_link.STL
- link left_shoulder_yaw_link: geometry collision cylinder length=0.024 radius=0.028; collision cylinder length=0.05 radius=0.042
- link left_wrist_pitch_link: geometry visual mesh filename=./meshes/left_wrist_pitch_link.STL
- link left_wrist_roll_link: geometry collision box size=0.07 0.045 0.14; visual mesh filename=./meshes/left_wrist_roll_link.STL
- link rgb_head_center: geometry visual mesh filename=./meshes/rgb_head_center_Link.STL
- link rgb_head_rear: geometry visual mesh filename=./meshes/rgb_head_rear_Link.STL
- link rgbd_head_front: geometry visual mesh filename=./meshes/rgbd_head_front_Link.STL
- link right_ankle_pitch_link: geometry visual mesh filename=./meshes/right_ankle_pitch_link.STL
- link right_ankle_roll_link: geometry collision sphere radius=0.005; collision sphere radius=0.005
- link right_elbow_link: geometry collision cylinder length=0.09 radius=0.04; visual mesh filename=./meshes/right_elbow_link.STL
- link right_hip_pitch_link: geometry visual mesh filename=./meshes/right_hip_pitch_link.STL
- link right_hip_yaw_link: geometry collision cylinder length=0.03 radius=0.042; collision cylinder length=0.03 radius=0.042
- link right_shoulder_pitch_link: geometry visual mesh filename=./meshes/right_shoulder_pitch_link.STL
- link right_shoulder_yaw_link: geometry collision cylinder length=0.024 radius=0.028; collision cylinder length=0.05 radius=0.042
- link right_wrist_pitch_link: geometry visual mesh filename=./meshes/right_wrist_pitch_link.STL
- link right_wrist_roll_link: geometry collision box size=0.07 0.045 0.14; visual mesh filename=./meshes/right_wrist_roll_link.STL
- link stereo_head_front: geometry visual mesh filename=./meshes/stereo_head_front_Link.STL
Joints:
- removed joint base_link_joint
- removed joint lidar_chest_front
